File: main/_autosave-main.kicad_pcb (KiCad board)
At the start: 2 copper layers, 30 x 95 mm, 38 parts, among them J1 Conn_Eurorack_5, U1 TL072, U2 TL072

Commit message: V2.0
Routing:
- net GND: track 0.00 -> 278.0 mm, vias 0 -> 3
- net +12V: track 0.00 -> 136.0 mm, vias 0 -> 3
- net Net-(OUT2-PadT): track 0.00 -> 88.4 mm, vias 0 -> 1
- net Net-(ATTACK1-Pad2): track 0.00 -> 87.5 mm, vias 0 -> 2
- net Net-(OUT1-PadT): track 0.00 -> 80.0 mm, vias 0 -> 1
- net Net-(D3-Pad1): track 0.00 -> 75.8 mm
- net Net-(IN2-PadT): track 0.00 -> 67.9 mm
- net Net-(ATTACK2-Pad2): track 0.00 -> 64.4 mm, vias 0 -> 1
- net Net-(D5-Pad1): track 0.00 -> 59.6 mm
- net -12V: track 0.00 -> 50.9 mm, vias 0 -> 1
- net Net-(IN1-PadT): track 0.00 -> 50.1 mm, vias 0 -> 1
- net Net-(D3-Pad2): track 0.00 -> 49.5 mm
- net Net-(D1-Pad1): track 0.00 -> 46.7 mm, vias 0 -> 2
- net Net-(R6-Pad2): track 0.00 -> 46.4 mm, vias 0 -> 3
- net Net-(D8-Pad2): track 0.00 -> 45.7 mm, vias 0 -> 2
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Other:
- board text added: "LMNC 2x AR ENV V2.0"
- board text removed: "LMNC 2x AR ENV V1.0"
